File: Hardware/Digital_resistor/AD5235.kicad_sch (KiCad schematic)
At the start: 5 parts, among them J1 Conn_02x03, U1 AD5235BRUZ250-R7

Commit message: finish layout
Parts:
- renumbered J1 to J6, U1 to U6
Connections:
- net R0-B: now reaches J6.1 (+12V), U6.6 (A1)
- net R1-B: now reaches J6.2 (+12V), U6.11 (A2)
- net R0-W: now reaches J6.3 (GND), U6.7 (W1)
- net R1-W: now reaches J6.4 (GND), U6.10 (W2)
- net R0-A: now reaches J6.5 (GND), U6.8 (B1)
- net R1-A: now reaches J6.6 (GND), U6.9 (B2)
Changed lines of the file:
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@@
     (stroke (width 0) (type default))
+  )
+  (label "R1-W" (at 142.24 135.89 0) (fields_autoplaced)
+    (effects (font (size 1.27 1.27)) (justify left bottom))
+  )
+  (label "R0-W" (at 116.84 135.89 0) (fields_autoplaced)
+    (effects (font (size 1.27 1.27)) (justify left bottom))
+  )
+  (label "R1-A" (at 142.24 133.35 0) (fields_autoplaced)
+    (effects (font (size 1.27 1.27)) (justify left bottom))
+  )
+  (label "R0-B" (at 116.84 138.43 0) (fields_autoplaced)
+    (effects (font (size 1.27 1.27)) (justify left bottom))
+  )
+  (label "R1-B" (at 142.24 138.43 0) (fields_autoplaced)
+    (effects (font (size 1.27 1.27)) (justify left bottom))
+  )
+  (label "R0-A" (at 116.84 133.35 0) (fields_autoplaced)
+    (effects (font (size 1.27 1.27)) (justify left bottom))
   )
   (hierarchical_label "SDI" (shape input) (at 76.2 74.93 180) (fields_autoplaced)
@@
   (symbol (lib_id "PCM_4ms_Connector:Conn_02x03") (at 133.35 135.89 0) (mirror x) (unit 1)
     (in_bom yes) (on_board yes) (dnp no)
-    (property "Reference" "J1" (at 133.35 144.78 0)
+    (property "Reference" "J6" (at 133.35 144.78 0)
       (effects (font (size 1.27 1.27)))
     )
@@
       (project "Digital_resistor"
         (path "/39961e6f-a344-457f-bf77-17001d2372f3/acf9be93-9339-4dc4-83a8-8ca1057885a4"
-          (reference "J1") (unit 1)
+          (reference "J6") (unit 1)
         )
         (path "/39961e6f-a344-457f-bf77-17001d2372f3/7e5db31c-6d0d-4589-b40d-85994497e35f"
+          (reference "J4") (unit 1)
+        )
+        (path "/39961e6f-a344-457f-bf77-17001d2372f3/04dd5ef7-d041-41b1-8272-c3dbae7efcd3"
           (reference "J2") (unit 1)
         )
-        (path "/39961e6f-a344-457f-bf77-17001d2372f3/04dd5ef7-d041-41b1-8272-c3dbae7efcd3"
-          (reference "J3") (unit 1)
-        )
         (path "/39961e6f-a344-457f-bf77-17001d2372f3/1ede5d6d-d221-46b5-9ca7-f7eccbe58a54"
-          (reference "J4") (unit 1)
+          (reference "J0") (unit 1)
         )
       )
@@
   (symbol (lib_id "Analog_local:AD5235BRUZ250-R7") (at 134.62 87.63 0) (unit 1)
     (in_bom yes) (on_board yes) (dnp no) (fields_autoplaced)
-    (property "Reference" "U1" (at 134.62 57.15 0)
+    (property "Reference" "U6" (at 134.62 57.15 0)
       (effects (font (size 1.27 1.27)))
     )
@@
       (project "Digital_resistor"
         (path "/39961e6f-a344-457f-bf77-17001d2372f3/acf9be93-9339-4dc4-83a8-8ca1057885a4"
-          (reference "U1") (unit 1)
+          (reference "U6") (unit 1)
         )
         (path "/39961e6f-a344-457f-bf77-17001d2372f3/7e5db31c-6d0d-4589-b40d-85994497e35f"
+          (reference "U4") (unit 1)
+        )
+        (path "/39961e6f-a344-457f-bf77-17001d2372f3/1ede5d6d-d221-46b5-9ca7-f7eccbe58a54"
+          (reference "U0") (unit 1)
+        )
+        (path "/39961e6f-a344-457f-bf77-17001d2372f3/04dd5ef7-d041-41b1-8272-c3dbae7efcd3"
           (reference "U2") (unit 1)
         )
-        (path "/39961e6f-a344-457f-bf77-17001d2372f3/1ede5d6d-d221-46b5-9ca7-f7eccbe58a54"
-          (reference "U4") (unit 1)
-        )
-        (path "/39961e6f-a344-457f-bf77-17001d2372f3/04dd5ef7-d041-41b1-8272-c3dbae7efcd3"
-          (reference "U3") (unit 1)
-        )
       )
