File: Hardware/Digital_resistor/mech.kicad_sch (KiCad schematic)
At the start: 4 parts

Commit message: finish layout
Parts:
- added H5, H6: MountingHole, MountingHole:MountingHole_3.2mm_M3_ISO14580, symbol Mechanical:MountingHole
Changed lines of the file:
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@@
+    )
+  )
+  (symbol (lib_id "Mechanical:MountingHole") (at 67.31 125.73 0) (unit 1)
+    (in_bom yes) (on_board yes) (dnp no) (fields_autoplaced)
+    (property "Reference" "H6" (at 69.85 124.46 0)
+      (effects (font (size 1.27 1.27)) (justify left))
+    )
+    (property "Value" "MountingHole" (at 69.85 127 0)
+      (effects (font (size 1.27 1.27)) (justify left))
+    )
+    (property "Footprint" "MountingHole:MountingHole_3.2mm_M3_ISO14580" (at 67.31 125.73 0)
+      (effects (font (size 1.27 1.27)) hide)
+    )
+    (property "Datasheet" "~" (at 67.31 125.73 0)
+      (effects (font (size 1.27 1.27)) hide)
+    )
+    (instances
+      (project "Digital_resistor"
+        (path "/39961e6f-a344-457f-bf77-17001d2372f3/d037a6d1-505b-4969-b3bc-675c82011bd0"
+          (reference "H6") (unit 1)
+        )
+      )
+    )
+  )
+  (symbol (lib_id "Mechanical:MountingHole") (at 67.31 119.38 0) (unit 1)
+    (in_bom yes) (on_board yes) (dnp no) (fields_autoplaced)
+    (property "Reference" "H5" (at 69.85 118.11 0)
+      (effects (font (size 1.27 1.27)) (justify left))
+    )
+    (property "Value" "MountingHole" (at 69.85 120.65 0)
+      (effects (font (size 1.27 1.27)) (justify left))
+    )
+    (property "Footprint" "MountingHole:MountingHole_3.2mm_M3_ISO14580" (at 67.31 119.38 0)
+      (effects (font (size 1.27 1.27)) hide)
+    )
+    (property "Datasheet" "~" (at 67.31 119.38 0)
+      (effects (font (size 1.27 1.27)) hide)
+    )
+    (instances
+      (project "Digital_resistor"
+        (path "/39961e6f-a344-457f-bf77-17001d2372f3/d037a6d1-505b-4969-b3bc-675c82011bd0"
+          (reference "H5") (unit 1)
+        )
+      )
     )
   )
