File: Hardware/Digital_resistor/rp2040-zero.kicad_sch (KiCad schematic)
At the start: 17 parts, among them SW5 SW_Push, SW6 SW_Push, SW7 SW_Push, SW8 SW_Push, U7 M24C02-WMN

Commit message: finish layout
Parts:
- added C11, C12, C13, C14, C15, C16, C17: 100nF_0603_16V, PCM_4ms_Capacitor:C_0603, symbol PCM_4ms_Capacitor:100nF_0603_16V
- added J1: Micro_SD_Card_Det2, Connectors_local:J_SD_Card-micro_socket_A, symbol Connectors_local:Micro_SD_Card_Det2
- added J7: Conn_01x03, PCM_4ms_Connector:Pins_1x03_2.54mm_TH_AudioInsRGndL, symbol PCM_4ms_Connector:Conn_01x03
- added R5, R6: 4.7k_0603, PCM_4ms_Resistor:R_0603, symbol PCM_4ms_Resistor:4.7k_0603
- added U5: ~, Boards:SSD1306-0.91-OLED-4pin-128x32, symbol Boards:0.91inchOled_32x128
- renumbered SW5 to SW1, SW6 to SW2, SW7 to SW3, SW8 to SW4
Connections:
- net +3V3: now also C11.1, C13.1, J1.4 (VDD), J7.1 (Pin_1), R5.1, R6.1, U5.2 (Vin)
- net +5V: now also RZ1.23 (+5V), C12.1, J7.3 (Pin_3); no longer RZ1.22 (5V)
- net GND: now also RZ1.22 (GND), C11.2, C12.2, C13.2, C14.2, C15.2, C16.2, C17.2, J1.6 (VSS), J1.SH (SHIELD), J7.2 (Pin_2), U5.1 (GND); no longer RZ1.23 (GND)
- net MISO: now also RZ1.9 (GP8); no longer RZ1.5 (GP4)
- net MOSI: now also RZ1.12 (GP11); no longer RZ1.4 (GP3)
- net RDY: now also RZ1.13 (GP12); no longer RZ1.8 (GP7)
- net SCK: now also RZ1.11 (GP10); no longer RZ1.7 (GP6)
- net SS: now also RZ1.10 (GP9); no longer RZ1.6 (GP5)
- net at R15.2, SW1.2: now also RZ1.16 (GP15), C17.1; no longer RZ1.15 (GP14)
- net at R16.2, SW2.2: now also RZ1.17 (GP26), C16.1; no longer RZ1.16 (GP15)
- net at R17.2, SW3.2: now also RZ1.19 (GP28), C15.1; no longer RZ1.17 (GP26)
- net at R18.2, RZ1.18 (GP27), SW4.2: now also C14.1
- net SPI0_SCK: now reaches RZ1.3 (GP2)
- net SPI0_SCK: now also J1.5 (CLK)
- new net I2C1_SCL: R5.2, RZ1.8 (GP7), U5.3 (SCK)
- new net I2C1_SDA: R6.2, RZ1.7 (GP6), U5.4 (SDA)
- new net SPI0_CS: J1.2 (DAT3/CD), RZ1.6 (GP5)
- new net SPI0_RX: J1.7 (DAT0), RZ1.5 (GP4)
- new net SPI0_TX: J1.3 (CMD), RZ1.4 (GP3)
- no-connect marks 7 -> 4
Other:
- note added: "SD card slot Raspberry Pi Pico DAT2 (NC) DAT3/CS ----- GP17 (SPI0 CSn) (Pin 22) CMD /DI ----- GP19 (SPI0 TX - MOSI) (Pin 25) VDD ----- 3V3 OUT (Pin 36) CLK/SCK ----- GP18 (SPI0 SCK) (Pin 24) VSS ----- GND (Pin 3 or 38 or ...) DAT0/DO ----- GP16 (SPI0 RX - MISO) (Pin 21) DAT1 (NC)"
- moved on the sheet: C9, R10, R11, R12, R15, R16, R17, R18, SW1, SW2, SW3, SW4
