File: Hardware/Digital_resistor/Digital_resistor.kicad_pcb (KiCad board)
At the start: 2 copper layers, 60 x 46 mm, 36 parts, among them J1 Conn_02x03, J2 Conn_02x03, J3 Conn_02x03, J4 Conn_02x03, SW1 SW_Push, SW2 SW_Push, SW3 SW_Push, SW4 SW_Push, U1 AD5235BRUZ250-R7, U2 AD5235BRUZ250-R7, U3 AD5235BRUZ250-R7, U4 AD5235BRUZ250-R7, U6 M24C02-WMN

Commit message: finish layout
Parts:
- removed A1: Arduino_Nano_Every, Boards:Arduino_Nano
- removed R7, R8, R9: 10k_0603_0.1%, PCM_4ms_Resistor:R_0603
- removed the U6 at (101.8, 59.9)
- added C10: 100nF_0603_16V, PCM_4ms_Capacitor:C_0603, F.Cu at (121.2, 41.4)
- added C11: 100nF_0603_16V, PCM_4ms_Capacitor:C_0603, B.Cu at (101.5, 52.8)
- added C12: 100nF_0603_16V, PCM_4ms_Capacitor:C_0603, B.Cu at (90.8, 53.0)
- added C13: 100nF_0603_16V, PCM_4ms_Capacitor:C_0603, B.Cu at (90.8, 56.3)
- added C14: 100nF_0603_16V, PCM_4ms_Capacitor:C_0603, B.Cu at (85.0, 48.2)
- added C15: 100nF_0603_16V, PCM_4ms_Capacitor:C_0603, B.Cu at (85.0, 58.5)
- added C16: 100nF_0603_16V, PCM_4ms_Capacitor:C_0603, B.Cu at (85.0, 68.1)
- added C17: 100nF_0603_16V, PCM_4ms_Capacitor:C_0603, B.Cu at (85.0, 78.2)
- added C9: 100nF_0603_16V, PCM_4ms_Capacitor:C_0603, B.Cu at (97.3, 61.0)
- added H5: MountingHole, MountingHole:MountingHole_3.2mm_M3_ISO14580, F.Cu at (137.0, 38.0)
- added H6: MountingHole, MountingHole:MountingHole_3.2mm_M3_ISO14580, F.Cu at (137.0, 87.0)
- added J1: Micro_SD_Card_Det2, Connectors_local:J_SD_Card-micro_socket_A, B.Cu at (101.6, 43.0)
- added J5: Conn_02x05_Odd_Even, Connector_PinHeader_2.54mm:PinHeader_2x05_P2.54mm_Vertical, F.Cu at (97.2, 85.2)
- added J7: Conn_01x03, PCM_4ms_Connector:Pins_1x03_2.54mm_TH_AudioInsRGndL, F.Cu at (92.2, 84.8)
- added R10: 10k_0603_0.1%, PCM_4ms_Resistor:R_0603, B.Cu at (97.3, 55.7)
- added R11: 10k_0603_0.1%, PCM_4ms_Resistor:R_0603, B.Cu at (97.3, 57.4)
- added R12: 10k_0603_0.1%, PCM_4ms_Resistor:R_0603, B.Cu at (97.3, 59.2)
- added R13: 4.7k_0603, PCM_4ms_Resistor:R_0603, B.Cu at (106.2, 52.3)
- added R14: 4.7k_0603, PCM_4ms_Resistor:R_0603, B.Cu at (106.2, 54.1)
- added R15: 10k_0603_0.1%, PCM_4ms_Resistor:R_0603, B.Cu at (97.3, 68.1)
- added R16: 10k_0603_0.1%, PCM_4ms_Resistor:R_0603, B.Cu at (97.3, 66.3)
- added R17: 10k_0603_0.1%, PCM_4ms_Resistor:R_0603, B.Cu at (97.3, 62.8)
- added R18: 10k_0603_0.1%, PCM_4ms_Resistor:R_0603, B.Cu at (97.3, 64.6)
- added REF**: OSHW-Logo2_9.8x8mm_SilkScreen, Symbol:OSHW-Logo2_9.8x8mm_SilkScreen, B.Cu at (135.9, 67.7)
- added REF**: KiCad-Logo2_6mm_SilkScreen, Symbol:KiCad-Logo2_6mm_SilkScreen, B.Cu at (135.1, 51.7)
- added RZ1: RP2040-Zero, Boards:RP2040-Zero, F.Cu at (91.3, 74.5)
- added U7: M24C02-WMN, Package_SO:SOIC-8_3.9x4.9mm_P1.27mm, F.Cu at (117.6, 39.8)
- R1, R2, R3: value 10k_0603_0.1% -> 2.2k_0603; moved to F.Cu
- R4: value 4.7k_0603 -> 2.2k_0603; moved to F.Cu
- R6: value 10k_0603_0.1% -> 4.7k_0603; moved to B.Cu
- moved R6 42.6 mm to (104.8, 67.3)
- moved U5 38.3 mm to (102.7, 42.2), turned to -90 degrees
- moved SW1 32.8 mm to (88.2, 80.5), turned to 180 degrees
- moved R3 28.5 mm to (115.6, 50.4), turned to -90 degrees
- moved R4 25.2 mm to (115.8, 85.1), turned to 90 degrees
- moved SW4 22.2 mm to (88.2, 50.5), turned to 180 degrees
- moved R2 16.6 mm to (114.1, 60.3), turned to -90 degrees
- moved SW2 15.3 mm to (88.2, 70.5), turned to 180 degrees
- moved R1 14.0 mm to (114.2, 70.1), turned to -90 degrees
- moved H1 10.3 mm to (128.0, 87.0)
- moved H4 10.3 mm to (128.0, 38.0)
- moved R5 9.65 mm to (104.8, 69.1)
- moved SW3 6.38 mm to (88.2, 60.5), turned to 180 degrees
- moved H2 5.00 mm to (83.0, 87.0)
- moved H3 5.00 mm to (83.0, 38.0)
- renumbered J4 to J0, J3 to J2, J2 to J4, J1 to J6, U4 to U0, U3 to U2, U2 to U4, U1 to U6
Connections:
- net /AD5235-1/CLK renamed /CPU_RP2040-zero/SPI1_SCK
- net /AD5235-1/CS renamed /CPU_RP2040-zero/SPI1_CS
- net Net-(A1-SCL/A5) renamed /CPU_RP2040-zero/I2C1_SCL
- net Net-(U1-A1) renamed /AD5235-1/R0-B
- net Net-(U1-A2) renamed /AD5235-1/R1-B
- net Net-(U1-B1) renamed /AD5235-1/R0-A
- net Net-(U1-B2) renamed /AD5235-1/R1-A
- net Net-(U1-W1) renamed /AD5235-1/R0-W
- net Net-(U1-W2) renamed /AD5235-1/R1-W
- net Net-(U2-A1) renamed /AD5235-2/R0-B
- net Net-(U2-A2) renamed /AD5235-2/R1-B
- net Net-(U2-B1) renamed /AD5235-2/R0-A
- net Net-(U2-B2) renamed /AD5235-2/R1-A
- net Net-(U2-W1) renamed /AD5235-2/R0-W
- net Net-(U2-W2) renamed /AD5235-2/R1-W
- net Net-(U3-A1) renamed /AD5235-3/R0-B
- net Net-(U3-A2) renamed /AD5235-3/R1-B
- net Net-(U3-B1) renamed /AD5235-3/R0-A
- net Net-(U3-B2) renamed /AD5235-3/R1-A
- net Net-(U3-W1) renamed /AD5235-3/R0-W
- net Net-(U3-W2) renamed /AD5235-3/R1-W
- net Net-(U4-A1) renamed /AD5235-4/R0-B
- net Net-(U4-A2) renamed /AD5235-4/R1-B
- net Net-(U4-B1) renamed /AD5235-4/R0-A
- net Net-(U4-B2) renamed /AD5235-4/R1-A
- net Net-(U4-W1) renamed /AD5235-4/R0-W
- net Net-(U4-W2) renamed /AD5235-4/R1-W
- R1 pad 2: /CPU/AI_P5V -> /AD5235-1/SDO
- R2 pad 1: /CPU/AI_P5V -> +5V
- R2 pad 2: GND -> /AD5235-2/SDO
- R3 pad 2: /AD5235-1/RDY -> /AD5235-3/SDO
- R4 pad 2: Net-(A1-SDA/A4) -> /CPU_RP2040-zero/SPI1_TX
- R5 pad 1: +5V -> +3V3
- R6 pad 1: +5V -> +3V3
- R6 pad 2: Net-(A1-D2) -> /CPU_RP2040-zero/I2C1_SDA
- SW1 pad 2: Net-(A1-D2) -> Net-(RZ1-GP15)
- U0 pad 16: /AD5235-1/RDY -> /CPU_RP2040-zero/AD_RDY
- U0 pad 3: /AD5235-4/SDO -> /CPU_RP2040-zero/SPI1_TX
- U2 pad 16: /AD5235-1/RDY -> /CPU_RP2040-zero/AD_RDY
- U4 pad 16: /AD5235-1/RDY -> /CPU_RP2040-zero/AD_RDY
- U5 pad 2: +5V -> +3V3
- U5 pad 4: Net-(A1-SDA/A4) -> /CPU_RP2040-zero/I2C1_SDA
- U6 pad 16: /AD5235-1/RDY -> /CPU_RP2040-zero/AD_RDY
- U6 pad 2: /AD5235-1/SDI -> /CPU_RP2040-zero/SPI1_RX
Routing:
- net +3V3: track 0.00 -> 109.8 mm, vias 0 -> 3
- net /AD5235-1/RDY: track 78.6 -> 0.00 mm, vias 4 -> 0
- net /CPU_RP2040-zero/AD_RDY: track 0.00 -> 71.4 mm, vias 0 -> 1
- net /CPU_RP2040-zero/SPI1_TX: track 0.00 -> 68.8 mm, vias 0 -> 3
- net /AD5235-4/SDO: track 56.3 -> 0.00 mm, vias 1 -> 0
- net +5V: track 133.7 -> 185.5 mm, vias 7 -> 5
- net GND: track 3.43 -> 43.6 mm, vias 1 -> 63
- net Net-(RZ1-GP27): track 0.00 -> 39.7 mm
- net /CPU_RP2040-zero/I2C1_SDA: track 0.00 -> 35.7 mm
- net /CPU_RP2040-zero/SPI1_RX: track 0.00 -> 30.0 mm, vias 0 -> 1
- net /AD5235-1/SDI: track 28.6 -> 0.00 mm, vias 1 -> 0
- net /CPU_RP2040-zero/I2C1_SCL: track 2.39 -> 29.6 mm
- net Net-(RZ1-GP15): track 0.00 -> 23.1 mm
- net Net-(RZ1-GP28): track 0.00 -> 23.0 mm
- net /CPU_RP2040-zero/SPI1_SCK: track 46.5 -> 69.0 mm, vias 4 -> 5
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- added copper zone on B.Cu, net GND
- added copper zone on F.Cu, net GND
Other:
- board size 60 x 46 mm -> 60 x 55 mm
- board text added: "0"
- board text added: "1"
- board text added: "15"
- board text added: "2"
- board text added: "2024"
- board text added: "26"
- board text added: "27"
- board text added: "28"
- board text added: "29"
- board text added: "3"
- board text added: "3V3"
- board text added: "3v3"
- board text added: "4"
- board text added: "5"
- board text added: "5V"
- board text added: "6"
- board text added: "7"
- board text added: "9"
- board text added: "Adwark"
- board text added: "Digital resistor V1"
- board text added: "GND"
- board text added: "R0B R0W R0A"
- board text added: "R1B R1W R1A"
- board text added: "R2B R2W R2A"
- board text added: "R3B R3W R3A"
- board text added: "R4B R4W R4A"
- board text added: "R5B R5W R5A"
- board text added: "R6B R6W R6A"
- board text added: "R7B R7W R7A"
- board text added: "achestni@visteon.com"
- board text added: "https://github.com/ami3go"

Commit message: Added Gerbers
Other:
- board text added: "AD5235"
- board text added: "M24C02"
Changed lines of the file:
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@@
     )
   )
+  (gr_circle (center 137 87) (end 139.202272 87)
+    (stroke (width 0.25) (type default)) (fill none) (layer "F.SilkS"))
+  (gr_circle (center 137 38) (end 139.202272 38)
+    (stroke (width 0.25) (type default)) (fill none) (layer "F.SilkS"))
+  (gr_circle (center 128 87) (end 130.202272 87)
+    (stroke (width 0.25) (type default)) (fill none) (layer "F.SilkS"))
+  (gr_circle (center 128 38) (end 130.202272 38)
+    (stroke (width 0.25) (type default)) (fill none) (layer "F.SilkS"))
+  (gr_circle (center 83 87) (end 85.202272 87)
+    (stroke (width 0.25) (type default)) (fill none) (layer "F.SilkS"))
+  (gr_circle (center 83 38) (end 85.202272 38)
+    (stroke (width 0.25) (type default)) (fill none) (layer "F.SilkS"))
   (gr_line (start 80 35) (end 80 90)
     (stroke (width 0.1) (type default)) (layer "Edge.Cuts"))
@@
     (effects (font (size 1 1) (thickness 0.15)) (justify left bottom))
   )
+  (gr_text "AD5235" (at 117.2 71.2) (layer "F.SilkS")
+    (effects (font (size 0.8 0.8) (thickness 0.2) bold) (justify left bottom))
+  )
   (gr_text "5" (at 106.9 65) (layer "F.SilkS" knockout)
     (effects (font (size 1 1) (thickness 0.15)) (justify left bottom))
@@
     (effects (font (size 1 1) (thickness 0.15)) (justify left bottom))
   )
+  (gr_text "AD5235" (at 117.2 61) (layer "F.SilkS")
+    (effects (font (size 0.8 0.8) (thickness 0.2) bold) (justify left bottom))
+  )
   (gr_text "29" (at 95.1 59.9) (layer "F.SilkS" knockout)
     (effects (font (size 1 1) (thickness 0.15)) (justify left bottom))
@@
     (effects (font (size 1.2 1.2) (thickness 0.3) bold) (justify left bottom))
   )
+  (gr_text "AD5235" (at 117.3 81) (layer "F.SilkS")
+    (effects (font (size 0.8 0.8) (thickness 0.2) bold) (justify left bottom))
+  )
   (gr_text "5V" (at 94.9 52.4) (layer "F.SilkS" knockout)
     (effects (font (size 1 1) (thickness 0.15)) (justify left bottom))
   )
+  (gr_text "M24C02" (at 115.04 40.775) (layer "F.SilkS")
+    (effects (font (size 0.8 0.8) (thickness 0.2) bold) (justify left bottom))
+  )
+  (gr_text "AD5235" (at 117.2 50.8) (layer "F.SilkS")
+    (effects (font (size 0.8 0.8) (thickness 0.2) bold) (justify left bottom))
+  )
   (gr_text "0" (at 106.6 52.4) (layer "F.SilkS" knockout)
