File: Hardware/Digital_resistor_v2/Digital_resistor.kicad_pcb (KiCad board)
At the start: 2 copper layers, 60 x 55 mm, 58 parts, among them J0 Conn_02x03, J1 Micro_SD_Card_Det2, J10 Conn_01x03, J2 Conn_02x03, J3 Conn_01x03, J4 Conn_02x03, J5 Conn_02x05_Odd_Even, J6 Conn_02x03, J7 Conn_01x03, J8 Conn_01x03, J9 Conn_01x03, SW1 SW_Push, SW2 SW_Push, SW3 SW_Push, SW4 SW_Push, U0 AD5235BRUZ250-R7, U2 AD5235BRUZ250-R7, U4 AD5235BRUZ250-R7, U6 AD5235BRUZ250-R7

Commit message: capture working state
Parts:
- moved R4 4.65 mm to (113.8, 80.9), turned to -90 degrees
Connections:
- net /AD5235-1/SDO renamed /SDO1-SDI2
- net /AD5235-2/SDO renamed /SDO2-SDI3
- net /AD5235-3/SDO renamed /SDO3-SDI4
- J5 pad 5: /CPU_RP2040-zero/SPI1_TX -> /CPU_RP2040-zero/SPI1_RX
- J5 pad 8: /CPU_RP2040-zero/SPI1_RX -> /CPU_RP2040-zero/SPI1_TX
- R4 pad 2: /CPU_RP2040-zero/SPI1_TX -> /CPU_RP2040-zero/SPI1_RX
- U0 pad 3: /CPU_RP2040-zero/SPI1_TX -> /CPU_RP2040-zero/SPI1_RX
- U6 pad 2: /CPU_RP2040-zero/SPI1_RX -> /CPU_RP2040-zero/SPI1_TX
Routing:
- net /CPU_RP2040-zero/SPI1_TX: track 68.8 -> 29.8 mm, vias 3 -> 0
- net /CPU_RP2040-zero/SPI1_RX: track 30.0 -> 65.2 mm, vias 1 -> 3
- net /CPU_RP2040-zero/SPI1_SCK: track 69.0 -> 72.2 mm, vias 5 -> 4
- net +5V: track 185.9 -> 187.3 mm
- net /CPU_RP2040-zero/AD_RDY: track 71.4 -> 70.8 mm
- net /CPU_RP2040-zero/SPI1_CS: track 77.6 -> 77.7 mm, vias 1 -> 2
